File: vhf_uhf_Diplexer_10W.kicad_pcb (KiCad board)
At the start: 2 copper layers, 57.1 x 44.5 mm, 17 parts, among them J1 3mm mount, J2 3mm mount, J3 3mm mount, J4 3mm mount, P1 SMA, P2 SMA, P3 SMA

Commit message: adding pdf dokumets
Parts:
- moved L1 0.64 mm to (52.7, 48.3)
- moved L2 0.64 mm to (66.7, 48.3), turned to 270 degrees
- moved C1 0.63 mm to (59.7, 50.2)
- moved C2 0.63 mm to (74.9, 50.2)
Routing:
- net GND: track 0.00 -> 172.7 mm
- net Net-(C3-Pad2): track 0.00 -> 18.8 mm
- net Net-(C2-Pad1): track 0.00 -> 13.6 mm
- net Net-(C4-Pad1): track 0.00 -> 12.5 mm
- net Net-(C1-Pad1): track 0.00 -> 11.5 mm
- net Net-(C3-Pad1): track 0.00 -> 11.3 mm
- net Net-(L3-Pad1): track 0.00 -> 10.2 mm
- net Net-(C5-Pad1): track 0.00 -> 6.89 mm
- added copper zone on B.Cu, net GND
- added copper zone on F.Cu, net GND
Other:
- board outline removed
- net class 50Ohm added: clearance 0.27, trace_width 1.6, via_dia 0.6, via_drill 0.4
